Commit message: modified

File: quadruped_robot_description/urdf/quadruped_robot.urdf (robot description, URDF)
Before this commit: robot quadruped_robot, 4 links, 3 joints
Links:
- removed link link1
- removed link link2
- added link gear_2, mass 0.8505876351103128; collision mesh filename=package://quadruped_robot_description/meshes/gear_2.stl scale=0.001 0.001 0.001; visual mesh filename=package://quadruped_robot_description/meshes/gear_2.stl scale=0.001 0.001 0.001
- added link leg_1, mass 0.8145141492777322; collision mesh filename=package://quadruped_robot_description/meshes/leg_1.stl scale=0.001 0.001 0.001; visual mesh filename=package://quadruped_robot_description/meshes/leg_1.stl scale=0.001 0.001 0.001
- added link leg_2, mass 2.0086761793539414; collision mesh filename=package://quadruped_robot_description/meshes/leg_2.stl scale=0.001 0.001 0.001; visual mesh filename=package://quadruped_robot_description/meshes/leg_2.stl scale=0.001 0.001 0.001
- added link leg_3, mass 0.657885902828282; collision mesh filename=package://quadruped_robot_description/meshes/leg_3.stl scale=0.001 0.001 0.001; visual mesh filename=package://quadruped_robot_description/meshes/leg_3.stl scale=0.001 0.001 0.001
- link base_link: mass 0.8505876350848196 -> 0.8505876351103128
Joints:
- removed joint revolute_1
- removed joint revolute_2
- added joint fixed1: type fixed, parent leg_3, child gear_2, origin xyz=0.0 -0.024 -0.0 rpy=0 0 0
- added joint fixed2: type fixed, parent gear_2, child leg_2, origin xyz=0.0 -0.025 0.0 rpy=0 0 0
- added joint revolute1: type revolute, parent base_link, child leg_3, origin xyz=0.0 0.025 0.0 rpy=0 0 0, axis 0.0 -1.0 0.0, limit lower=-3.141592 upper=3.141592 effort=50 velocity=20.0
- added joint revolute2: type revolute, parent leg_2, child leg_1, origin xyz=0.190612 -0.02 -0.11005 rpy=0 0 0, axis 0.0 -1.0 -0.0, limit lower=-3.141592 upper=3.141592 effort=50 velocity=20.0
